File: hardware/transmitter/SerialTransmitter.kicad_pcb (KiCad board)
At the start: 2 copper layers, 78.7 x 70.5 mm, 42 parts, among them J1 Conn_01x08_Male, J2 Conn_01x02_Male, J3 Conn_01x03_Male, J4 Conn_01x08_Male, J5 Conn_01x03_Male, J6 Conn_01x04_Male, Q1 2N7000, SW1 SW_DIP_x08, SW2 SW_Push, U1 74LS165, U2 74LS191, U3 74LS74, U4 74LS132, U5 74LS132, U6 74LS244

Commit message: Added some notes to the schematic, changed the names of the components, moved some parts.
Parts:
- J1: value Conn_01x08_Male -> DATA
- J2: value Conn_01x02_Male -> OUTPUT
- J4: value Conn_01x08_Male -> Control
- J6: value Conn_01x04_Male -> CLK_SELECT
- U1: value 74LS165 -> 74HC165
- U3: value 74LS74 -> 74HC74
- U4, U5: value 74LS132 -> 74HC132
- U6: value 74LS244 -> 74HC244
Changed lines of the file:
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@@
   (net 42 "Net-(U5-Pad1)")
   (net 43 "Net-(J4-Pad5)")
-  (net 44 "Net-(J4-Pad8)")
+  (net 44 "Net-(R7-Pad2)")
   (net 45 "Net-(C7-Pad1)")
   (net 46 "Net-(RV1-Pad3)")
-  (net 47 "Net-(U1-Pad2)")
+  (net 47 "Net-(J6-Pad2)")
   (net 48 "Net-(D1-Pad2)")
   (net 49 "Net-(D2-Pad2)")
@@
   (net 51 "Net-(D3-Pad2)")
   (net 52 "Net-(J2-Pad2)")
-  (net 53 "Net-(U4-Pad11)")
+  (net 53 "Net-(J6-Pad3)")
   (footprint "Capacitor_THT:C_Disc_D3.0mm_W2.0mm_P2.50mm" (layer "F.Cu")
     (at 168.315 71.775)
@@
       (effects (font (size 1 1) (thickness 0.15)))
     )
-    (fp_text value "Conn_01x08_Male" (at 4.385 20.05) (layer "F.Fab")
+    (fp_text value "Control" (at 4.385 20.05) (layer "F.Fab")
       (effects (font (size 1 1) (thickness 0.15)))
     )
@@
       (net 40 "unconnected-(J4-Pad7)") (pinfunction "Pin_7") (pintype "passive"))
     (pad "8" thru_hole oval (at 0 17.78 180) (size 1.7 1.7) (drill 1) (layers *.Cu *.Mask)
-      (net 44 "Net-(J4-Pad8)") (pinfunction "Pin_8") (pintype "passive"))
+      (net 44 "Net-(R7-Pad2)") (pinfunction "Pin_8") (pintype "passive"))
     (model "${KICAD6_3DMODEL_DIR}/Connector_PinHeader_2.54mm.3dshapes/PinHeader_1x08_P2.54mm_Horizontal.wrl"
       (offset (xyz 0 0 0))
@@
       (effects (font (size 1 1) (thickness 0.15)))
     )
-    (fp_text value "74LS165" (at 3.81 20.11) (layer "F.Fab")
+    (fp_text value "74HC165" (at 3.81 20.11) (layer "F.Fab")
       (effects (font (size 1 1) (thickness 0.15)))
     )
@@
       (net 4 "Net-(U1-Pad1)") (pinfunction "~{PL}") (pintype "input"))
     (pad "2" thru_hole oval (at 0 2.54) (size 1.6 1.6) (drill 0.8) (layers *.Cu *.Mask)
-      (net 47 "Net-(U1-Pad2)") (pinfunction "CP") (pintype "input"))
+      (net 47 "Net-(J6-Pad2)") (pinfunction "CP") (pintype "input"))
     (pad "3" thru_hole oval (at 0 5.08) (size 1.6 1.6) (drill 0.8) (layers *.Cu *.Mask)
       (net 20 "/D3") (pinfunction "D4") (pintype "input"))
@@
       (effects (font (size 1 1) (thickness 0.15)))
     )
-    (fp_text value "74LS244" (at 3.81 25.19) (layer "F.Fab")
+    (fp_text value "74HC244" (at 3.81 25.19) (layer "F.Fab")
       (effects (font (size 1 1) (thickness 0.15)))
     )
@@
       (effects (font (size 1 1) (thickness 0.15)))
     )
-    (fp_text value "Conn_01x02_Male" (at 4.385 4.81 90) (layer "F.Fab")
+    (fp_text value "OUTPUT" (at 4.385 4.81 90) (layer "F.Fab")
       (effects (font (size 1 1) (thickness 0.15)))
     )
@@
       (net 49 "Net-(D2-Pad2)") (pintype "passive"))
     (pad "2" thru_hole oval (at 10.16 0 180) (size 1.6 1.6) (drill 0.8) (layers *.Cu *.Mask)
-      (net 44 "Net-(J4-Pad8)") (pintype "passive"))
+      (net 44 "Net-(R7-Pad2)") (pintype "passive"))
     (model "${KICAD6_3DMODEL_DIR}/Resistor_THT.3dshapes/R_Axial_DIN0207_L6.3mm_D2.5mm_P10.16mm_Horizontal.wrl"
       (offset (xyz 0 0 0))
@@
       (net 1 "GND") (pintype "passive"))
     (pad "2" thru_hole oval (at 10.16 0 270) (size 1.6 1.6) (drill 0.8) (layers *.Cu *.Mask)
-      (net 47 "Net-(U1-Pad2)") (pintype "passive"))
+      (net 47 "Net-(J6-Pad2)") (pintype "passive"))
     (model "${KICAD6_3DMODEL_DIR}/Resistor_THT.3dshapes/R_Axial_DIN0207_L6.3mm_D2.5mm_P10.16mm_Horizontal.wrl"
       (offset (xyz 0 0 0))
@@
       (effects (font (size 1 1) (thickness 0.15)))
     )
-    (fp_text value "Conn_01x08_Male" (at 4.385 20.05) (layer "F.Fab")
+    (fp_text value "DATA" (at 4.385 20.05) (layer "F.Fab")
       (effects (font (size 1 1) (thickness 0.15)))
     )
@@
       (effects (font (size 1 1) (thickness 0.15)))
     )
-    (fp_text value "Conn_01x04_Male" (at 0 9.95) (layer "F.Fab")
+    (fp_text value "CLK_SELECT" (at 0 9.95) (layer "F.Fab")
       (effects (font (size 1 1) (thickness 0.15)))
     )
@@
       (net 1 "GND") (pinfunction "Pin_1") (pintype "passive"))
     (pad "2" thru_hole oval (at 0 2.54 180) (size 1.7 1.7) (drill 1) (layers *.Cu *.Mask)
-      (net 47 "Net-(U1-Pad2)") (pinfunction "Pin_2") (pintype "passive"))
+      (net 47 "Net-(J6-Pad2)") (pinfunction "Pin_2") (pintype "passive"))
     (pad "3" thru_hole oval (at 0 5.08 180) (size 1.7 1.7) (drill 1) (layers *.Cu *.Mask)
-      (net 53 "Net-(U4-Pad11)") (pinfunction "Pin_3") (pintype "passive"))
+      (net 53 "Net-(J6-Pad3)") (pinfunction "Pin_3") (pintype "passive"))
     (pad "4" thru_hole oval (at 0 7.62 180) (size 1.7 1.7) (drill 1) (layers *.Cu *.Mask)
-      (net 53 "Net-(U4-Pad11)") (pinfunction "Pin_4") (pintype "passive"))
+      (net 53 "Net-(J6-Pad3)") (pinfunction "Pin_4") (pintype "passive"))
     (model "${KICAD6_3DMODEL_DIR}/Connector_PinHeader_2.54mm.3dshapes/PinHeader_1x04_P2.54mm_Vertical.wrl"
       (offset (xyz 0 0 0))
@@
       (effects (font (size 1 1) (thickness 0.15)))
     )
-    (fp_text value "74LS132" (at 3.81 17.57) (layer "F.Fab")
+    (fp_text value "74HC132" (at 3.81 17.57) (layer "F.Fab")
       (effects (font (size 1 1) (thickness 0.15)))
     )
@@
       (net 45 "Net-(C7-Pad1)") (pintype "input"))
     (pad "11" thru_hole oval (at 7.62 7.62) (size 1.6 1.6) (drill 0.8) (layers *.Cu *.Mask)
-      (net 53 "Net-(U4-Pad11)") (pintype "output"))
+      (net 53 "Net-(J6-Pad3)") (pintype "output"))
     (pad "12" thru_hole oval (at 7.62 5.08) (size 1.6 1.6) (drill 0.8) (layers *.Cu *.Mask)
       (net 46 "Net-(RV1-Pad3)") (pintype "input"))
@@
       (net 14 "unconnected-(U2-Pad13)") (pinfunction "Rc") (pintype "output"))
     (pad "14" thru_hole oval (at 7.62 5.08) (size 1.6 1.6) (drill 0.8) (layers *.Cu *.Mask)
-      (net 47 "Net-(U1-Pad2)") (pinfunction "Cp") (pintype "input"))
+      (net 47 "Net-(J6-Pad2)") (pinfunction "Cp") (pintype "input"))
     (pad "15" thru_hole oval (at 7.62 2.54) (size 1.6 1.6) (drill 0.8) (layers *.Cu *.Mask)
       (net 1 "GND") (pinfunction "P0") (pintype "input"))
@@
       (effects (font (size 1 1) (thickness 0.15)))
     )
-    (fp_text value "74LS132" (at 3.81 17.57) (layer "F.Fab")
+    (fp_text value "74HC132" (at 3.81 17.57) (layer "F.Fab")
       (effects (font (size 1 1) (thickness 0.15)))
     )
@@
       (net 41 "Net-(U3-Pad6)") (pintype "input"))
     (pad "3" thru_hole oval (at 0 5.08) (size 1.6 1.6) (drill 0.8) (layers *.Cu *.Mask)
-      (net 44 "Net-(J4-Pad8)") (pintype "output"))
+      (net 44 "Net-(R7-Pad2)") (pintype "output"))
     (pad "4" thru_hole oval (at 0 7.62) (size 1.6 1.6) (drill 0.8) (layers *.Cu *.Mask)
       (net 43 "Net-(J4-Pad5)") (pintype "input"))
@@
       (effects (font (size 1 1) (thickness 0.15)))
     )
-    (fp_text value "74LS74" (at 3.81 17.57) (layer "F.Fab")
+    (fp_text value "74HC74" (at 3.81 17.57) (layer "F.Fab")
       (effects (font (size 1 1) (thickness 0.15)))
     )
@@
       (net 24 "Net-(U3-Pad2)") (pinfunction "D") (pintype "input"))
     (pad "3" thru_hole oval (at 0 5.08) (size 1.6 1.6) (drill 0.8) (layers *.Cu *.Mask)
-      (net 47 "Net-(U1-Pad2)") (pinfunction "C") (pintype "input"))
+      (net 47 "Net-(J6-Pad2)") (pinfunction "C") (pintype "input"))
     (pad "4" thru_hole oval (at 0 7.62) (size 1.6 1.6) (drill 0.8) (layers *.Cu *.Mask)
       (net 8 "VCC") (pinfunction "~{S}") (pintype "input"))
@@
       (net 8 "VCC") (pinfunction "~{S}") (pintype "input"))
     (pad "11" thru_hole oval (at 7.62 7.62) (size 1.6 1.6) (drill 0.8) (layers *.Cu *.Mask)
-      (net 47 "Net-(U1-Pad2)") (pinfunction "C") (pintype "input"))
+      (net 47 "Net-(J6-Pad2)") (pinfunction "C") (pintype "input"))
     (pad "12" thru_hole oval (at 7.62 5.08) (size 1.6 1.6) (drill 0.8) (layers *.Cu *.Mask)
       (net 26 "Net-(U3-Pad12)") (pinfunction "D") (pintype "input"))
